File: PacMan/Pacman2020.sch (KiCad schematic (older format))
At the start: 13 parts, among them J10 Conn_01x02, J11 Conn_01x02, J12 Conn_01x02, J13 Conn_01x08, J5 Conn_01x04, J9 Conn_01x02, Q2 Q_NMOS_GDS

Commit message: add parts note
Other:
- note added: "TODO: \nJ9-J12 need different part (2.5mm spacing B2B XH?)\nHV single pin connect need different part (DF-22)"
- note added: "Use 2.5mm spacing"
Changed lines of the file:
@@
 Wire Wire Line
 	5375 7375 6075 7375
+Text Notes 11000 4100 1    50   ~ 0
+Use 2.5mm spacing
+Text Notes 7100 6950 0    50   ~ 0
+TODO: \nJ9-J12 need different part (2.5mm spacing B2B XH?)\nHV single pin connect need different part (DF-22)
 $EndSCHEMATC
